Commit message: Se agrega launch de gráficas con plotjuggler y rviz, además se resuelven incompatibilidades del bumper sensor y lidar con rviz.

File: ros2_ws/src/peter_robot/urdf/peter.urdf.xacro (robot description, xacro)
@@ -74,5 +74,5 @@
             </lidar>
             <topic>scan</topic>
-            <gz_frame_id>laser_frame</gz_frame_id>
+            <gz_frame_id>lidar_link</gz_frame_id>
         </sensor>
     </gazebo>

File: ros2_ws/src/peter_robot/urdf/peter_control_plugin.xacro (robot description, xacro)
@@ -209,4 +209,29 @@
             <state_interface name="effort" />
         </joint>
+        <!-- Bumpers -->
+        <joint name="BumperRU_joint">
+            <command_interface name="position"/>
+            <state_interface name="position"/>
+            <state_interface name="velocity"/>
+            <state_interface name="effort"/>
+        </joint>
+        <joint name="BumperLU_joint">
+            <command_interface name="position"/>
+            <state_interface name="position"/>
+            <state_interface name="velocity"/>
+            <state_interface name="effort"/>
+        </joint>
+        <joint name="BumperRD_joint">
+            <command_interface name="position"/>
+            <state_interface name="position"/>
+            <state_interface name="velocity"/>
+            <state_interface name="effort"/>
+        </joint>
+        <joint name="BumperLD_joint">
+            <command_interface name="position"/>
+            <state_interface name="position"/>
+            <state_interface name="velocity"/>
+            <state_interface name="effort"/>
+        </joint>
     </ros2_control>
     <!-- LIMITES JOINTS -->
