Commit message: Se pulió la lógica de movimiento omnidireccional mediante algoritmo de control proporcional acotado junto con nuevas posiciones en el modo omnidireccional.

File: ros2_ws/src/peter_robot/urdf/peter.urdf (robot description, URDF)
Before this commit: robot Peter_3.0_completo, 26 links, 25 joints
Joints:
- joint CoxisLU_joint: limit lower=-1.13 upper=2 effort=200 velocity=200 -> lower=-1.57 upper=2 effort=200 velocity=200

Commit message: NUEVO URDF CON CEROS ACTUALIZADOS

File: ros2_ws/src/peter_robot/urdf/peter.urdf (robot description, URDF)
Before this commit: robot Peter_3.0_completo, 26 links, 25 joints
Links:
- link BumperLD_link: geometry collision box size=0.02 0.02 0.01; visual box size=0.02 0.02 0.01
- link BumperLU_link: geometry collision box size=0.02 0.02 0.01; visual box size=0.02 0.02 0.01
- link BumperRD_link: geometry collision box size=0.02 0.02 0.01; visual box size=0.02 0.02 0.01
- link BumperRU_link: geometry collision box size=0.02 0.02 0.01; visual box size=0.02 0.02 0.01
- link CoxisLD_link: mass 0.0515847132031574 -> 0.0515847008737883
- link CoxisLU_link: mass 0.0515847042228037 -> 0.0515847008737884
- link CoxisRD_link: mass 0.0515847017813385 -> 0.0515846904005967
- link CoxisRU_link: mass 0.0515847056526637 -> 0.0515846904005967
- link FemurLD_link: mass 0.0322370081893243 -> 0.0322370452082158
- link FemurLU_link: mass 0.0322370074530517 -> 0.0322370452082159
- link FemurRD_link: mass 0.0322370091635994 -> 0.0322370452082158
- link FemurRU_link: mass 0.0322370098830192 -> 0.0322370452082158
- link Head_z_link: mass 0.0103184369301582 -> 0.0103184370744868
- link RuedaLD_link: mass 0.0410439695671941 -> 0.041043969465079
- link RuedaLU_link: mass 0.0410439695181042 -> 0.0410439694650791
- link RuedaRD_link: mass 0.0410439698241763 -> 0.0410439694654469
- link RuedaRU_link: mass 0.0410439694665572 -> 0.041043969465447
- link TibiaLD_link: mass 0.0667476309214474 -> 0.0667476307461011
- link TibiaLU_link: mass 0.0667476310976818 -> 0.066747630746101
- link TibiaRD_link: mass 0.0667714118308176 -> 0.0667714120865956
- link TibiaRU_link: mass 0.0667714115678162 -> 0.0667714120865957
Joints:
- joint BumperLD_joint: origin xyz=0.14 -0.012938 -0.028054 rpy=0 0 0 -> xyz=0 0 0.03207 rpy=0 0 0; parent TibiaLD_link -> RuedaLD_link
- joint BumperLU_joint: origin xyz=0.14 -0.00459051118128878 -0.0302190306176173 rpy=0 0 0 -> xyz=0 0 0.03207 rpy=0 0 0; parent TibiaLU_link -> RuedaLU_link
- joint BumperRD_joint: origin xyz=0.14 -0.00138265547481653 0.0287708901417234 rpy=0 0 0 -> xyz=0 0 0.03207 rpy=0 0 0; parent TibiaRD_link -> RuedaRD_link
- joint BumperRU_joint: origin xyz=0.14 -0.0076711055817173 0.0283762200987518 rpy=0 0 0 -> xyz=0 0 0.03207 rpy=0 0 0; parent TibiaRU_link -> RuedaRU_link
- joint CoxisLD_joint: limit lower=-1.13 upper=2 effort=200 velocity=200 -> lower=-1.57 upper=1.57 effort=200 velocity=200
- joint CoxisLU_joint: limit lower=-1.57 upper=2 effort=200 velocity=200 -> lower=-1.57 upper=1.57 effort=200 velocity=200; origin xyz=0.096588 0.060798 -0.0098 rpy=-3.1416 0 1.5708 -> xyz=0.0965884887784687 0.060798386550441 -0.00979999999999995 rpy=-3.14159265358979 0 1.5707963267949
- joint CoxisRD_joint: limit lower=-2 upper=1.57 effort=200 velocity=200 -> lower=-1.57 upper=1.57 effort=200 velocity=200; origin xyz=-0.09323 -0.060798 -0.0098 rpy=3.1416 0 -1.5708 -> xyz=-0.0932301097293624 -0.0607983865504415 -0.00980000000000016 rpy=3.14159265358979 0 -1.5707963267949
- joint CoxisRU_joint: limit lower=-2 upper=1.57 effort=200 velocity=200 -> lower=-1.57 upper=1.57 effort=200 velocity=200; origin xyz=0.096588 -0.060798 -0.0098 rpy=3.1416 0 -1.5708 -> xyz=0.096588488778468 -0.0607983865504415 -0.00980000000000016 rpy=3.14159265358979 0 -1.5707963267949
- joint FemurLD_joint: axis 0.10217 0 0.99477 -> 0.70711 0 0.70711; limit lower=-2.8 upper=0.35 effort=200 velocity=200 -> lower=-1.57 upper=1.57 effort=200 velocity=200; origin xyz=0.046435 0.021468 -0.015752 rpy=-1.5708 0 0 -> xyz=0.049567 -0.012656 -0.015752 rpy=-1.5708 0 0
- joint FemurLU_joint: axis -0.1455 0 0.98936 -> -0.707106781186545 0 0.70710678118655; limit lower=-2.8 upper=0.35 effort=200 velocity=200 -> lower=-1.57 upper=1.57 effort=200 velocity=200; origin xyz=0.039628 0.032261 -0.015752 rpy=-1.5708 0 0 -> xyz=0.0125512915293921 0.0496036868635676 -0.0157518633540368 rpy=-1.5707963267949 0 0
- joint FemurRD_joint: axis 0.11804 0 -0.99301 -> 0.707106781186557 0 -0.707106781186538; limit lower=-0.35 upper=2.8 effort=200 velocity=200 -> lower=-1.57 upper=1.57 effort=200 velocity=200; origin xyz=0.046773 -0.020724 -0.015752 rpy=-1.5708 0 0 -> xyz=0.0495681853611769 0.0126572113832391 -0.0157518633540372 rpy=-1.57079632679489 0 0
- joint FemurRU_joint: axis 0.051392 0 -0.99868 -> -0.707106781186547 0 -0.707106781186548; limit lower=-2.0 upper=2.8 effort=200 velocity=200 -> lower=-1.57 upper=1.57 effort=200 velocity=200; origin xyz=0.045319 -0.0237 -0.015752 rpy=-1.5708 0 0 -> xyz=0.0126930684475665 -0.0494626210692686 -0.0157517010851108 rpy=-1.57079632679489 0 0
- joint Head_y_joint: axis 0.113197942878959 -0.993572456204363 0 -> 0 -1 0; origin xyz=0.00481057280523833 0.013430874479555 0.00994999999999966 rpy=0 0 0 -> xyz=0.00629999999999953 0.0128 0.00994999999999965 rpy=0 0 0
- joint RuedaLD_joint: axis 0.0033463 0.03258 -0.99946 -> 0 0 -1; origin xyz=0.10926 -0.012938 -0.028054 rpy=0 1.5708 0 -> xyz=0.109530068824489 -0.0252082867118495 -0.0161284884758471 rpy=0 1.5707963267949 0
- joint RuedaLU_joint: axis -0.0033473808290709 0.0227609837826761 -0.999735331304656 -> 0 0 -1; origin xyz=0.109353047449084 -0.00459051118128878 -0.0302190306176173 rpy=0 1.5707963267949 0 -> xyz=0.10953 0.016128 -0.025208 rpy=0 1.5708 0
- joint RuedaRD_joint: axis 0.00903692524308548 -0.0760217790170896 -0.997065205037879 -> 0 0 -1; origin xyz=0.109696793417255 -0.00138265547481653 0.0287708901417234 rpy=0 1.5707963267949 0 -> xyz=0.109529744274998 -0.0248291866544958 0.0158053456421234 rpy=0 1.5707963267949 0
- joint RuedaRU_joint: axis 8.35837727566709E-05 -0.00162426112226136 -0.999998677393905 -> 0 0 -1; origin xyz=0.109539977240268 -0.0076711055817173 0.0283762200987518 rpy=0 1.5707963267949 0 -> xyz=0.109529744274998 0.0158053456421239 0.0248291866544947 rpy=0 1.5707963267949 0
- joint TibiaLD_joint: axis 0 -0.10217 -0.99477 -> 0 -0.70711 -0.70711; limit lower=-2.7 upper=0.43 effort=200 velocity=200 -> lower=-2.38 upper=0.76 effort=200 velocity=200; origin xyz=0.062664 0.030509 -0.0064363 rpy=0 0 -1.5708 -> xyz=0.049493 0 -0.049493 rpy=0 0 -1.5708
- joint TibiaLU_joint: axis 0 0.1455 -0.98936 -> 0 0.70711 -0.70711; limit lower=-2.7 upper=0.43 effort=200 velocity=200 -> lower=-2.38 upper=0.76 effort=200 velocity=200; origin xyz=0.060661 0.033759 0.0089212 rpy=0 0 -1.5708 -> xyz=0.049493 0 0.049493 rpy=0 0 -1.5708
- joint TibiaRD_joint: axis 0 -0.11804 0.99301 -> 0 -0.70711 0.70711; limit lower=-0.43 upper=2.7 effort=200 velocity=200 -> lower=-0.76 upper=2.38 effort=200 velocity=200; origin xyz=0.056409 0.040891 0.0067056 rpy=0 0 -1.5708 -> xyz=0.049493 0 0.049493 rpy=0 0 -1.5708
- joint TibiaRU_joint: axis 0 -0.051392 0.99868 -> 0 0.707106781186552 0.707106781186543; limit lower=-0.43 upper=2.7 effort=200 velocity=200 -> lower=-0.76 upper=2.38 effort=200 velocity=200; origin xyz=0.06042 0.034948 0.0031092 rpy=0 0 -1.5708 -> xyz=0.0493513687238616 9.62765376531123E-05 -0.0493513687238616 rpy=0 0 -1.57079632679489

Commit message: Publicación de marcha mejorada y componentes de lidar test 1

File: ros2_ws/src/peter_robot/urdf/peter.urdf (robot description, URDF)
Before this commit: robot Peter_3.0_completo, 26 links, 25 joints
Links:
- link BumperLD_link: geometry collision box size=0.02 0.02 0.01; visual box size=0.005 0.005 0.0025
- link BumperLU_link: geometry collision box size=0.02 0.02 0.01; visual box size=0.005 0.005 0.0025
- link BumperRD_link: geometry collision box size=0.02 0.02 0.01; visual box size=0.005 0.005 0.0025
- link BumperRU_link: geometry collision box size=0.02 0.02 0.01; visual box size=0.005 0.005 0.0025

Commit message: Se realiza avances en movimiento omnidireccional, se plantean mejoras, tareas y además se graban resultados con gráficas de evasión de estímulo hostil

File: ros2_ws/src/peter_robot/urdf/peter.urdf (robot description, URDF)
Before this commit: robot Peter_3.0_completo, 26 links, 25 joints
Links:
- link RuedaLD_link: mass 0.0410439695671941 -> 0.410439695671941
- link RuedaLU_link: mass 0.0410439695181042 -> 0.410439695181042
- link RuedaRD_link: mass 0.0410439698241763 -> 0.410439698241763
- link RuedaRU_link: mass 0.0410439694665572 -> 0.410439694665572
